Commit message: feat: first gazebo simulation

File: description/robot.urdf.xacro (robot description, xacro)
@@ -2,3 +2,4 @@
 <robot xmlns:xacro="http://www.ros.org/wiki/xacro"  name="robot">
  <xacro:include filename="robot_core.xacro"/>
+ <xacro:include filename="gazebo_control.xacro"/>
 </robot>

File: description/robot_core.xacro (robot description, xacro)
@@ -86,4 +86,7 @@
         </xacro:inertial_cylinder>
     </link>
+    <gazebo reference="right_wheel">
+        <material>Gazebo/Blue</material>
+    </gazebo>
     <!-- CASTER WHEEL -->
     <joint name="caster_wheel_joint" type="fixed">
@@ -108,3 +111,7 @@
         </xacro:inertial_sphere>
     </link>
+    <gazebo reference="caster_wheel">
+        <mu1 value="0.0"/>
+        <mu2 value="0.0"/>
+    </gazebo>
 </robot>
